Commit message: UPDATE readme

File: src/gazebo_simulator/urdf/robot.xacro (robot description, xacro)
@@ -8,5 +8,6 @@
     <xacro:include filename="$(find gazebo_simulator)/urdf/depthCamera.xacro"/>
     <xacro:include filename="$(find gazebo_simulator)/urdf/ultraSound.xacro"/>
-    <xacro:include filename="$(find gazebo_simulator)/urdf/lidar.xacro"/>
+    <xacro:include filename="$(find gazebo_simulator)/urdf/vlp16_mount.xacro"/>
+    <!-- <xacro:include filename="$(find gazebo_simulator)/urdf/lidar.xacro"/> -->
     <!-- <xacro:stairs stairs="15" xpos="0" ypos="0" zpos="0" /> -->
     <!-- Rotor related joint and link is only for demonstrate location. -->
@@ -124,6 +125,9 @@
         <origin rpy="0 0 0" xyz="0.2747 0.0 -0.0088"/>
     </xacro:ultraSound>
-    <xacro:lidar parent="trunk">
+    <!-- <xacro:lidar parent="trunk">
         <origin rpy="0 0 0" xyz="0.05 0 0.08"/>
-    </xacro:lidar>
+    </xacro:lidar> -->
+    <xacro:vlp16_mount prefix="" parent_link="trunk" topic="velodyne_points" gpu="true">
+        <origin rpy="0 0 0" xyz="0.05 0 0.08"/>
+    </xacro:vlp16_mount>
 </robot>

Commit message: UPDATE scene setup

File: src/gazebo_simulator/urdf/robot.xacro (robot description, xacro)
@@ -128,5 +128,5 @@
         <origin rpy="0 0 0" xyz="0.05 0 0.08"/>
     </xacro:lidar> -->
-    <xacro:vlp16_mount prefix="" parent_link="trunk" topic="velodyne_points" gpu="true">
+    <xacro:vlp16_mount prefix="" parent_link="trunk" lidar_topic="velodyne_points" gpu="true">
         <origin rpy="0 0 0" xyz="0.05 0 0.08"/>
     </xacro:vlp16_mount>

File: src/gazebo_simulator/urdf/vlp16_mount.xacro (robot description, xacro)
@@ -2,5 +2,7 @@
 <robot xmlns:xacro="http://wiki.ros.org/xacro">
   <xacro:include filename="$(find velodyne_description)/urdf/VLP-16.urdf.xacro" />
-  <xacro:macro name="vlp16_mount" params="prefix parent_link topic gpu height:=0.12 *origin">
+  <xacro:include filename="$(find realsense2_description)/urdf/_d435.urdf.xacro" />
+  <xacro:arg name="use_nominal_extrinsics" default="false"/>
+  <xacro:macro name="vlp16_mount" params="prefix parent_link lidar_topic gpu height:=0.12 *origin">
     <!--
       The VLP16 is mounted to a pair of extrusion rods on top of the main sensor arch
@@ -78,7 +80,35 @@
       <origin xyz="0 0 ${height}" rpy="0 0 0"/>
     </joint>
-    <xacro:VLP-16 parent="${prefix}vlp16_mount_plate" topic="${topic}" gpu="${gpu}">
+    <xacro:VLP-16 parent="${prefix}vlp16_mount_plate" topic="${lidar_topic}" gpu="${gpu}">
       <origin xyz="0 0 0" rpy="0 0 0" />
     </xacro:VLP-16>
+    <!--
+      The D435 is mounted at the front of the main sensor arch
+    -->
+    <link name="${prefix}depth_camera_mount">
+      <visual>
+        <geometry>
+          <box size="0.04 0.04 0.02" />
+        </geometry>
+        <material name="black">
+          <color rgba="1 1 1 1" />
+        </material>
+        <origin xyz="0 0 0" rpy="0 0 0" />
+      </visual>
+      <collision>
+        <geometry>
+          <box size="0.04 0.04 0.02" />
+        </geometry>
+        <origin xyz="0 0 0" rpy="0 0 0" />
+      </collision>
+    </link>
+    <joint name="${prefix}depth_camera_mount_joint" type="fixed">
+      <parent link="${prefix}vlp16_mount_plate" />
+      <child link="${prefix}depth_camera_mount" />
+      <origin xyz="0.1 0 0" rpy="0 0 0" />
+    </joint>
+    <xacro:sensor_d435 name="camera" topics_ns="camera" parent="${prefix}depth_camera_mount" publish_pointcloud="true">
+      <origin xyz="0.02 0 -0.02" rpy="0 0 0" />
+    </xacro:sensor_d435>
   </xacro:macro>
 </robot>
